File: 1_PCB_RevA/LissajousRevA/LissajousRevA.brd (EAGLE design)
At the start: 99.1 x 66 mm, 77 parts, among them U101 LM348D, U201 LM348D, U401 LM348D

Commit message: Added silk and tidy up tracks
Routing:
- net V-: track 148.5 -> 122.5 mm
- net V+: track 257.9 -> 243.8 mm
- net 0V: track 308.5 -> 301.2 mm, vias 14 -> 13
- net N$20: track 49.4 -> 46.2 mm
- net N$16: track 29.3 -> 27.9 mm
- net N$25: track 59.5 -> 58.7 mm
- net N$17: track 41.4 -> 42.2 mm
- net N$38: track 136.3 -> 135.5 mm
- added copper zone on layer 16, net N$35
Other:
- board text added: "A1"
- board text added: "Ashley J. Robinson"
- board text added: "F1"
- board text added: "F2"
- board text added: "GND"
- board text added: "Jan 2016"
- board text added: "Lissajous"
- board text added: "P1"
- board text added: "RevA"
- board text added: "V+"
- board text added: "V-"
- board text added: "V1"
- board text added: "V2"

Commit message: flood and final tidy
Routing:
- net N$39: track 126.9 -> 78.4 mm, vias 2 -> 4
- net N$36: track 36.6 -> 34.4 mm
- net N$46: track 38.7 -> 40.5 mm
- net V-: track 122.5 -> 123.6 mm
- net 0V: track 301.2 -> 302.3 mm, vias 13 -> 14
- net N$37: vias 0 -> 2
- net N$12: vias 0 -> 2
- added copper zone on layer 16, net 0V
- added copper zone on layer 1, net V+
- added copper zone on layer 1, net V-
- removed copper zone on layer 16, net N$35
